File: kicad/pcba.kicad_pcb (KiCad board)
At the start: 2 copper layers, 74 x 37.5 mm, 27 parts, among them J1 Conn_01x02, J3 Conn_01x03_Pin, U1 TP4056-42-ESOP8, U2 TLV9062, U3 MCP4725xxx-xCH, U4 ESP32-C3-DevKitM-1, U5 AD8232ACPZ-R7, U7 TLV9062

Commit message: a
Parts:
- moved BT1 0.50 mm to (88.0, 148.0)
Changed lines of the file:
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@@
 	(footprint "Connector_JST:JST_PH_S2B-PH-K_1x02_P2.00mm_Horizontal"
 		(layer "F.Cu")
-		(at 87.55 148 90)
+		(at 88.05 148 90)
 		(descr "JST PH series connector, S2B-PH-K (http://www.jst-mfg.com/product/pdf/eng/ePH.pdf), generated with kicad-footprint-generator")
 		(tags "connector JST PH horizontal")
@@
 	)
 	(segment
+		(start 91 145.05)
+		(end 88.05 148)
+		(width 0.2)
+		(layer "F.Cu")
+		(net 33)
+	)
+	(segment
 		(start 87.499 134.904)
 		(end 87.499 132.82734)
@@
 	)
 	(segment
-		(start 91 144.55)
-		(end 91 142.5)
+		(start 91 142.5)
+		(end 91 145.05)
 		(width 0.2)
 		(layer "F.Cu")
@@
 	)
 	(segment
-		(start 87.55 148)
-		(end 91 144.55)
-		(width 0.2)
-		(layer "F.Cu")
-		(net 33)
-	)
-	(segment
 		(start 110.225 149.5)
 		(end 110.225 148.55)
@@
 	)
 	(segment
-		(start 87.55 146)
-		(end 87.55 140.645)
+		(start 87.92 140.275)
+		(end 87.92 145.87)
 		(width 0.2)
 		(layer "F.Cu")
@@
 	)
 	(segment
-		(start 87.55 140.645)
-		(end 87.92 140.275)
+		(start 87.92 145.87)
+		(end 88.05 146)
 		(width 0.2)
 		(layer "F.Cu")
